Commit message: se agrega tercer eslabon

File: src/dp/urdf/dp_base.xacro (robot description, xacro)
@@ -87,4 +87,28 @@
       </collision>
   </link>
+  <!-- Tercer eslabón -->
+  <!-- La terna 3 está en la entrada del eslabón => DH proximal  -->
+  <link name="link3">
+      <inertial>
+          <origin xyz="${a3/2.0} 0 0"/>
+          <mass value="${mass3}"/>
+          <inertia ixx="${ixx3}" ixy="0.0" ixz="0.0" iyy="${iyy3}" iyz="0.0" izz="${izz3}"/>
+      </inertial>
+      <visual>
+          <origin xyz="${a3/2.0} 0 0"/>
+          <geometry>
+              <box size="${length3} ${width3} ${width3}"/>
+          </geometry>
+          <material name="green">
+              <color rgba="0 1 0 1"/>
+          </material>
+      </visual>
+      <collision>
+          <origin xyz="${a3/2.0} 0 0"/>
+          <geometry>
+              <box size="${length3} ${width3} ${width3}"/>
+          </geometry>
+      </collision>
+  </link>
   <!--******************* DEFINICIONES DE JUNTAS  *******************-->
   <!-- Junta entre base y link1 -->
@@ -101,13 +125,22 @@
       <parent link="link1"/>
       <child link="link2"/>
-      <origin xyz="${a1} 0 ${width1}" rpy="0 0 0"/>
+      <origin xyz="${a2} 0 ${width2}" rpy="0 0 0"/>
       <axis xyz="0 0 1"/>
       <limit effort="$(arg tau2_max)" lower="$(arg q2_min)" upper="$(arg q2_max)" velocity="$(arg qp2_max)"/>
       <dynamics damping="$(arg damping2)" friction="$(arg friction2)"/>
   </joint>
+   <!-- Junta entre link2 y link3 -->
+  <joint name="joint3" type="revolute">
+      <parent link="link2"/>
+      <child link="link3"/>
+      <origin xyz="${a3} 0 ${width3}" rpy="0 0 0"/>
+      <axis xyz="0 0 1"/>
+      <limit effort="$(arg tau3_max)" lower="$(arg q3_min)" upper="$(arg q3_max)" velocity="$(arg qp3_max)"/>
+      <dynamics damping="$(arg damping3)" friction="$(arg friction3)"/>
+  </joint>
   <!--******************* DEFINICIONES DE HERRAMIENTA  *******************-->
   <!-- Terna TOOL0 en el extremo de link2 -->
   <joint name="tool0_joint" type="fixed">
-    <parent link="link2"/>
+    <parent link="link3"/>
     <child link="tool0"/>
     <origin xyz="${a2} 0 0" rpy="0 0 0"/>
@@ -135,4 +168,13 @@
     </joint>
   </transmission>
+  <transmission name="motor3_transmission">
+    <type>transmission_interface/SimpleTransmission</type>
+    <actuator name="motor3_actuator">
+      <mechanicalReduction>${N2}</mechanicalReduction>
+    </actuator>
+    <joint name="joint3">
+      <hardwareInterface>hardware_interface/PositionJointInterface</hardwareInterface>
+    </joint>
+  </transmission>
   <!--******************* CONFIGURACION DE ros2_control *******************-->
   <ros2_control name="GazeboSystem" type="system">
@@ -156,4 +198,19 @@
     </joint>
     <joint name="joint2">
+      <command_interface name="position">
+        <param name="min">-3.14</param>
+        <param name="max">3.14</param>
+      </command_interface>
+      <command_interface name="effort">
+        <param name="min">-100</param>
+        <param name="max">100</param>
+      </command_interface>
+      <state_interface name="position">
+        <param name="initial_value">$(arg q2_ini)</param>
+      </state_interface>
+      <state_interface name="velocity"/>
+      <state_interface name="effort"/>
+    </joint>
+    <joint name="joint3">
       <command_interface name="position">
         <param name="min">-3.14</param>

File: src/dp/urdf/dp_caos.xacro (robot description, xacro)
@@ -6,4 +6,6 @@
   <xacro:arg name="damping2" default="0.000001"/>              <!-- rozamiento viscoso -->
   <xacro:arg name="friction2" default="0.000001"/>             <!-- rozamiento de Coulomb -->
+  <xacro:arg name="damping3" default="0.000001"/>              <!-- rozamiento viscoso -->
+  <xacro:arg name="friction3" default="0.000001"/>             <!-- rozamiento de Coulomb -->
   <xacro:arg name="q1_max" default="3140.0"/>                  <!-- límite físico superior eje 1 -->
   <xacro:arg name="q1_min" default="-3140.0"/>                 <!-- límite físico inferior eje 1 -->
@@ -14,6 +16,11 @@
   <xacro:arg name="qp2_max" default="500.0"/>                  <!-- límite físico velocidad eje 2 -->
   <xacro:arg name="tau2_max" default="10000.0"/>               <!-- límite físico del esfuerzo aplicable en eje 2 -->
+  <xacro:arg name="q3_max" default="3140.0"/>                  <!-- límite físico superior eje 3 -->
+  <xacro:arg name="q23min" default="-3140.0"/>                 <!-- límite físico inferior eje 3 -->
+  <xacro:arg name="qp3_max" default="500.0"/>                  <!-- límite físico velocidad eje 3 -->
+  <xacro:arg name="tau3_max" default="10000.0"/>               <!-- límite físico del esfuerzo aplicable en eje 3 -->
   <xacro:arg name="q1_ini" default="1.0"/>                     <!-- condición inicial de posición -->
   <xacro:arg name="q2_ini" default="1.0"/>                     <!-- condición inicial de posición -->
+  <xacro:arg name="q3_ini" default="1.0"/>                     <!-- condición inicial de posición -->
   <!-- Incluir el modelo base -->
   <xacro:include filename="$(find dp)/urdf/dp_base.xacro"/>

File: src/dp/urdf/dp_loose.xacro (robot description, xacro)
@@ -6,5 +6,7 @@
   <xacro:arg name="q2_max" default="3140.0"/>                  <!-- límite físico superior eje 2 -->
   <xacro:arg name="q2_min" default="-3140.0"/>                 <!-- límite físico inferior eje 2 -->
-  <xacro:arg name="dp_fixed" default="false"/>
+  <xacro:arg name="q3_max" default="3140.0"/>                  <!-- límite físico superior eje 2 -->
+  <xacro:arg name="q3_min" default="-3140.0"/>                 <!-- límite físico inferior eje 2 -->
+  <xacro:arg name="dp_fixed" default="true"/>
   <!-- Incluir el modelo base -->
   <xacro:include filename="$(find dp)/urdf/dp_base.xacro"/>

File: src/dp/urdf/dp_params.xacro (robot description, xacro)
@@ -34,4 +34,16 @@
   <xacro:property name="izz2" value="${(1.0/12.0) * mass2 * (length2 * length2 + width2 * width2) + Jm2_ef}"/> <!-- super simplificación a fines didácticos -->
   <xacro:property name="iyy2" value="${izz2}"/>
+ <!-- Parámetros del eslabón 3. Prisma de sección cuadrada y centro de masa en el centro -->
+  <xacro:property name="mass3" value="1.5"/>                    <!-- masa de la barra que modela el eslabón -->
+  <xacro:property name="length3" value="0.22"/>                 <!-- largo total -->
+  <xacro:property name="width3" value="0.02"/>                  <!-- ancho de la sección total -->
+  <xacro:property name="a3" value="${length3 - width3}"/>       <!-- distancia entre ejes -->
+  <xacro:property name="Jm3" value="0.0001"/>                   <!-- inercia del rotor del motor -->
+  <xacro:property name="N3"  value="10"/>                       <!-- relación de transmisión -->
+  <xacro:property name="Jm3_ef" value="${N3*N3 * Jm3}"/>        <!-- inercia del rotor reflejada al eje -->
+  <!-- Calculo de la inercia de una barra (con motor en eje de rotación) para orientación a lo largo del eje X -->
+  <xacro:property name="ixx3" value="${(1.0/6.0) * mass3 * (width3 * width3)}"/>
+  <xacro:property name="izz3" value="${(1.0/12.0) * mass3 * (length3 * length3 + width3 * width3) + Jm3_ef}"/> <!-- super simplificación a fines didácticos -->
+  <xacro:property name="iyy3" value="${izz3}"/>
   <!-- Valores que pueden modificarse en otros archivos xacro y que funcionan como argumentos -->
   <xacro:arg name="damping1" default="0.1"/>                 <!-- rozamiento viscoso -->
@@ -39,4 +51,6 @@
   <xacro:arg name="damping2" default="0.1"/>                 <!-- rozamiento viscoso -->
   <xacro:arg name="friction2" default="0.01"/>               <!-- rozamiento de Coulomb -->
+  <xacro:arg name="damping3" default="0.1"/>                 <!-- rozamiento viscoso -->
+  <xacro:arg name="friction3" default="0.01"/>               <!-- rozamiento de Coulomb -->
   <xacro:arg name="q1_max" default="3.14"/>                  <!-- límite físico superior eje 1 -->
   <xacro:arg name="q1_min" default="-3.14"/>                 <!-- límite físico inferior eje 1 -->
@@ -47,5 +61,10 @@
   <xacro:arg name="qp2_max" default="5.0"/>                  <!-- límite físico velocidad eje 2 -->
   <xacro:arg name="tau2_max" default="100.0"/>               <!-- límite físico del esfuerzo aplicable en eje 2 -->
+  <xacro:arg name="q3_max" default="3.14"/>                  <!-- límite físico superior eje 3 -->
+  <xacro:arg name="q3_min" default="-3.14"/>                 <!-- límite físico inferior eje 3 -->
+  <xacro:arg name="qp3_max" default="5.0"/>                  <!-- límite físico velocidad eje 3 -->
+  <xacro:arg name="tau3_max" default="100.0"/>               <!-- límite físico del esfuerzo aplicable en eje 3 -->
   <xacro:arg name="q1_ini" default="1.0"/>                   <!-- condición inicial de posición -->
   <xacro:arg name="q2_ini" default="1.0"/>                   <!-- condición inicial de posición -->
+  <xacro:arg name="q3_ini" default="1.0"/>                   <!-- condición inicial de posición -->
 </robot>

Commit message: variando cosas...

File: src/dp/urdf/dp_base.xacro (robot description, xacro)
@@ -125,5 +125,5 @@
       <parent link="link1"/>
       <child link="link2"/>
-      <origin xyz="${a2} 0 ${width2}" rpy="0 0 0"/>
+      <origin xyz="${a1} 0 ${width1}" rpy="0 0 0"/>
       <axis xyz="0 0 1"/>
       <limit effort="$(arg tau2_max)" lower="$(arg q2_min)" upper="$(arg q2_max)" velocity="$(arg qp2_max)"/>
@@ -134,5 +134,5 @@
       <parent link="link2"/>
       <child link="link3"/>
-      <origin xyz="${a3} 0 ${width3}" rpy="0 0 0"/>
+      <origin xyz="${a2} 0 ${width2}" rpy="0 0 0"/>
       <axis xyz="0 0 1"/>
       <limit effort="$(arg tau3_max)" lower="$(arg q3_min)" upper="$(arg q3_max)" velocity="$(arg qp3_max)"/>
@@ -140,9 +140,9 @@
   </joint>
   <!--******************* DEFINICIONES DE HERRAMIENTA  *******************-->
-  <!-- Terna TOOL0 en el extremo de link2 -->
+  <!-- Terna TOOL0 en el extremo de link3 -->
   <joint name="tool0_joint" type="fixed">
     <parent link="link3"/>
     <child link="tool0"/>
-    <origin xyz="${a2} 0 0" rpy="0 0 0"/>
+    <origin xyz="${a3} 0 0" rpy="0 0 0"/>
   </joint>
   <link name="tool0"/>
@@ -171,5 +171,5 @@
     <type>transmission_interface/SimpleTransmission</type>
     <actuator name="motor3_actuator">
-      <mechanicalReduction>${N2}</mechanicalReduction>
+      <mechanicalReduction>${N3}</mechanicalReduction>
     </actuator>
     <joint name="joint3">
@@ -222,5 +222,5 @@
       </command_interface>
       <state_interface name="position">
-        <param name="initial_value">$(arg q2_ini)</param>
+        <param name="initial_value">$(arg q3_ini)</param>
       </state_interface>
       <state_interface name="velocity"/>

File: src/dp/urdf/dp_params.xacro (robot description, xacro)
@@ -2,5 +2,5 @@
 <robot xmlns:xacro="http://www.ros.org/wiki/xacro">
   <!-- Parámetros del eslabón 0. Cilindro y centro de masa en el centro -->
-  <xacro:property name="mass0" value="1.5"/>
+  <xacro:property name="mass0" value="15"/>
   <xacro:property name="radius0" value="0.05"/> <!-- largo total -->
   <xacro:property name="height0" value="0.04"/>
@@ -24,5 +24,5 @@
   <!-- Parámetros del eslabón 2. Prisma de sección cuadrada y centro de masa en el centro -->
   <xacro:property name="mass2" value="1.5"/>                    <!-- masa de la barra que modela el eslabón -->
-  <xacro:property name="length2" value="0.22"/>                 <!-- largo total -->
+  <xacro:property name="length2" value="0.165"/>                 <!-- largo total -->
   <xacro:property name="width2" value="0.02"/>                  <!-- ancho de la sección total -->
   <xacro:property name="a2" value="${length2 - width2}"/>       <!-- distancia entre ejes -->
@@ -36,5 +36,5 @@
  <!-- Parámetros del eslabón 3. Prisma de sección cuadrada y centro de masa en el centro -->
   <xacro:property name="mass3" value="1.5"/>                    <!-- masa de la barra que modela el eslabón -->
-  <xacro:property name="length3" value="0.22"/>                 <!-- largo total -->
+  <xacro:property name="length3" value="0.11"/>                 <!-- largo total -->
   <xacro:property name="width3" value="0.02"/>                  <!-- ancho de la sección total -->
   <xacro:property name="a3" value="${length3 - width3}"/>       <!-- distancia entre ejes -->
